File: body/cad/leds/leds.sch (KiCad schematic (older format))
At the start: 38 parts

Commit message: first pcb steps
Parts:
- added J1: Conn_01x02, Pin_Headers:Pin_Header_Straight_1x02_Pitch2.54mm, symbol Conn_01x02
- D1, D10, D11, D12, D13, D14, D15, D16, D17, D18, D19, D2, D20, D21, D22, D23, D24, D25, D26, D27, D28, D29, D3, D30, D31, D32, D33, D34, D35, D36, D4, D5, D6, D7, D8, D9: renamed from D?; footprint (none) -> LEDs:LED_D5.0mm
- SW1: renamed from SW?; footprint (none) -> Buttons_Switches_ThroughHole:SW_DIP_x2_W7.62mm_Piano
Connections:
- net +3V8: now also SW1.3 (A), J1.1 (Pin_1); no longer SW1.1 (A)
- net GND: now also J1.2 (Pin_2)
- net at D10.2 (A), D13.2 (A), D14.2 (A)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: now also SW1.4 (B); no longer SW1.2 (B)

Commit message: optimze design, finalize layout
Parts:
- removed SW1: SW_DPST_x2, Buttons_Switches_ThroughHole:SW_DIP_x2_W7.62mm_Piano, symbol SW_DPST_x2
- added J2: Conn_01x02, Pin_Headers:Pin_Header_Straight_1x02_Pitch2.54mm, symbol Conn_01x02
Connections:
- net +3V8 is gone; now on net Wide_Circle: J1.1 (Pin_1)
- net GND: now also J2.2 (Pin_2); no longer J1.2 (Pin_2)
- net Wide_Circle: now reaches D1.2 (A), D11.2 (A), D12.2 (A), D17.2 (A), D18.2 (A), D2.2 (A), D23.2 (A), D24.2 (A), D29.2 (A), D3.2 (A), D30.2 (A), D31.2 (A), D32.2 (A), D33.2 (A), D34.2 (A), D35.2 (A), D36.2 (A), D4.2 (A), D5.2 (A), D6.2 (A)
- net Spott_Circle: now reaches D10.2 (A), D13.2 (A), D14.2 (A), D15.2 (A), D16.2 (A), D19.2 (A), D20.2 (A), D21.2 (A), D22.2 (A), D25.2 (A), D26.2 (A), D27.2 (A), D28.2 (A), D7.2 (A), D8.2 (A), D9.2 (A)
- net Spott_Circle: now also J1.2 (Pin_2), J2.1 (Pin_1)
Changed lines of the file:
@@
 	1    0    0    -1
-$EndComp
-$Comp
-L +3V8 #PWR02
-U 1 1 5A2D8D76
-P 1400 4200
-F 0 "#PWR02" H 1400 4050 50  0001 C CNN
-F 1 "+3V8" H 1400 4340 50  0000 C CNN
-F 2 "" H 1400 4200 50  0001 C CNN
-F 3 "" H 1400 4200 50  0001 C CNN
-	1    1400 4200
-	-1   0    0    1
 $EndComp
 Wire Wire Line
@@
 	3800 1150 3800 2250
 Wire Wire Line
-	2200 3550 2200 1250
-Wire Wire Line
 	2200 1250 2850 1250
 Wire Wire Line
@@
 	1    0    0    -1
 $EndComp
+Wire Wire Line
+	1400 1050 1400 3000
 $Comp
-L SW_DPST_x2 SW1
-U 2 1 5A2D932A
-P 1400 3800
-F 0 "SW1" H 1400 3925 50  0000 C CNN
-F 1 "SW_DPST_x2" H 1400 3700 50  0000 C CNN
-F 2 "Buttons_Switches_ThroughHole:SW_DIP_x2_W7.62mm_Piano" H 1400 3800 50  0001 C CNN
-F 3 "" H 1400 3800 50  0001 C CNN
-	2    1400 3800
+L PWR_FLAG #FLG05
+U 1 1 5A2DA64F
+P 1100 3000
+F 0 "#FLG05" H 1100 3075 50  0001 C CNN
+F 1 "PWR_FLAG" H 900 3250 50  0000 C CNN
+F 2 "" H 1100 3000 50  0001 C CNN
+F 3 "" H 1100 3000 50  0001 C CNN
+	1    1100 3000
 	0    -1   -1   0
 $EndComp
+Text GLabel 1400 3000 2    60   Input ~ 0
+Wide_Circle
 Wire Wire Line
-	1400 3400 1400 3600
+	2200 3550 2200 1250
+Text GLabel 2200 3550 2    60   Input ~ 0
+Spott_Circle
+Text GLabel 1500 4150 0    60   Input ~ 0
+Spott_Circle
 $Comp
-L SW_DPST_x2 SW1
-U 1 1 5A2D9717
-P 1400 3200
-F 0 "SW1" H 1400 3325 50  0000 C CNN
-F 1 "SW_DPST_x2" H 1400 3100 50  0000 C CNN
-F 2 "Buttons_Switches_ThroughHole:SW_DIP_x2_W7.62mm_Piano" H 1400 3200 50  0001 C CNN
-F 3 "" H 1400 3200 50  0001 C CNN
-	1    1400 3200
-	0    -1   -1   0
-$EndComp
-Wire Wire Line
-	1400 1050 1400 3000
-Wire Wire Line
-	1400 3550 2200 3550
-Connection ~ 1400 3550
-Wire Wire Line
-	1400 4200 1400 4000
-$Comp
-L Conn_01x02 J1
-U 1 1 5A2D9D54
-P 2250 4100
-F 0 "J1" H 2250 4200 50  0000 C CNN
-F 1 "Conn_01x02" H 2600 4100 50  0000 C CNN
-F 2 "Pin_Headers:Pin_Header_Straight_1x02_Pitch2.54mm" H 2250 4100 50  0001 C CNN
-F 3 "" H 2250 4100 50  0001 C CNN
-	1    2250 4100
+L GND #PWR06
+U 1 1 5A2DDE55
+P 1500 4250
+F 0 "#PWR06" H 1500 4000 50  0001 C CNN
+F 1 "GND" H 1500 4100 50  0000 C CNN
+F 2 "" H 1500 4250 50  0001 C CNN
+F 3 "" H 1500 4250 50  0001 C CNN
+	1    1500 4250
 	1    0    0    -1
 $EndComp
 $Comp
-L GND #PWR04
-U 1 1 5A2D9DD1
-P 2050 4200
-F 0 "#PWR04" H 2050 3950 50  0001 C CNN
-F 1 "GND" H 2050 4050 50  0000 C CNN
-F 2 "" H 2050 4200 50  0001 C CNN
-F 3 "" H 2050 4200 50  0001 C CNN
-	1    2050 4200
+L Conn_01x02 J1
+U 1 1 5A2DF3DF
+P 1650 3650
+F 0 "J1" H 1650 3750 50  0000 C CNN
+F 1 "Conn_01x02" V 1800 3600 50  0000 C CNN
+F 2 "Pin_Headers:Pin_Header_Straight_1x02_Pitch2.54mm" H 1650 3650 50  0001 C CNN
+F 3 "" H 1650 3650 50  0001 C CNN
+	1    1650 3650
+	0    -1   -1   0
+$EndComp
+Text GLabel 1650 3850 0    60   Input ~ 0
+Wide_Circle
+Text GLabel 1750 3850 2    60   Input ~ 0
+Spott_Circle
+$Comp
+L Conn_01x02 J2
+U 1 1 5A2DF5A8
+P 1700 4150
+F 0 "J2" H 1700 4250 50  0000 C CNN
+F 1 "Conn_01x02" V 1850 4100 50  0000 C CNN
+F 2 "Pin_Headers:Pin_Header_Straight_1x02_Pitch2.54mm" H 1700 4150 50  0001 C CNN
+F 3 "" H 1700 4150 50  0001 C CNN
+	1    1700 4150
 	1    0    0    -1
 $EndComp
-$Comp
-L +3V8 #PWR05
-U 1 1 5A2D9ED9
-P 2050 4100
-F 0 "#PWR05" H 2050 3950 50  0001 C CNN
-F 1 "+3V8" H 2050 4240 50  0000 C CNN
-F 2 "" H 2050 4100 50  0001 C CNN
-F 3 "" H 2050 4100 50  0001 C CNN
-	1    2050 4100
-	1    0    0    -1
-$EndComp
-$Comp
-L PWR_FLAG #FLG06
-U 1 1 5A2DA5ED
-P 2050 4100
-F 0 "#FLG06" H 2050 4175 50  0001 C CNN
-F 1 "PWR_FLAG" H 2200 4350 50  0000 C CNN
-F 2 "" H 2050 4100 50  0001 C CNN
-F 3 "" H 2050 4100 50  0001 C CNN
-	1    2050 4100
-	0    -1   -1   0
-$EndComp
-$Comp
-L PWR_FLAG #FLG07
-U 1 1 5A2DA64F
-P 2050 4200
-F 0 "#FLG07" H 2050 4275 50  0001 C CNN
-F 1 "PWR_FLAG" H 1850 4450 50  0000 C CNN
-F 2 "" H 2050 4200 50  0001 C CNN
-F 3 "" H 2050 4200 50  0001 C CNN
-	1    2050 4200
-	0    -1   -1   0
-$EndComp
 $EndSCHEMATC
